Commit message: feat:更新参数

File: robobus_description/urdf/vehicle.xacro (robot description, xacro)
@@ -6,7 +6,7 @@
   <link name="base_link">
     <visual>
-      <origin xyz="-2.0 0.0 0.1" rpy="0 0 ${pi/2.0}"/>
+      <origin xyz="0.0 0.0 -0.4" rpy="0 0 0"/>
       <geometry>
-        <mesh filename="package://robobus_description/mesh/hooke.dae" scale="0.001 0.001 0.001"/>
+        <mesh filename="package://robobus_description/mesh/robobus.dae" scale="1.0 1.0 1.0"/>
       </geometry>
     </visual>

Commit message: feat: update urdf

File: robobus_description/urdf/vehicle.xacro (robot description, xacro)
@@ -6,5 +6,5 @@
   <link name="base_link">
     <visual>
-      <origin xyz="0.0 0.0 -0.4" rpy="0 0 0"/>
+      <origin xyz="0.0 0.1 -0.4" rpy="0 0 0"/>
       <geometry>
         <mesh filename="package://robobus_description/mesh/robobus.dae" scale="1.0 1.0 1.0"/>
